Commit message: add base footprint

File: description/urdf/diffbot_description.urdf.xacro (robot description, xacro)
@@ -14,4 +14,6 @@
   <xacro:property name="caster_wheel_radius" value="0.015" />
   <xacro:property name="z_offset" value="-${base_height/2}" /> <!-- Space btw top of beam and the each joint -->
+  <!-- Base_Footprint-->
+  <link name="${prefix}base_footprint"/>
   <!-- Base Link -->
   <link name="${prefix}base_link">

Commit message: add  base footprint joint

File: description/urdf/diffbot_description.urdf.xacro (robot description, xacro)
@@ -16,4 +16,9 @@
   <!-- Base_Footprint-->
   <link name="${prefix}base_footprint"/>
+  <joint name="${prefix}base_footprint_joint" type="fixed">
+      <parent link="${prefix}base_footprint"/>
+      <child link="${prefix}base_link"/>
+      <origin xyz="0 0 0" rpy="0 0 0"/>
+    </joint>
   <!-- Base Link -->
   <link name="${prefix}base_link">
